File: hardware/synthesizer/coxial_conn.kicad_sch (KiCad schematic)
At the start: 4 parts, among them J10 Output 2, J6 Input 1, J7 Input 2, J9 Output 1

Commit message: further improvements
Parts:
- added C?: 3mF, symbol Device:C
- added R15, R23, R26: 200k, symbol Device:R
- added R21, R25, R?: 10k, symbol Device:R
- added R24: 6.8k, symbol Device:R
- added R?: 4.7k, symbol Device:R
- added U7, U?: OPA196xDGK, Package_SO:VSSOP-8_3x3mm_P0.65mm, symbol Amplifier_Operational:OPA196xDGK
Connections:
- net GND: now also R23.1, R24.2
- net OUT_1: now reaches J9.1 (In)
- net OUT_1: now also R15.2, U7.6
- net IN_2: now reaches J7.1 (In)
- net IN_1: now reaches J6.1 (In)
- net OUT_2: now reaches J10.1 (In)
- new net: R15.1, R?.2, U7.2 (-)
- new net: R21.1, R23.2, U7.3 (+)
- new net +0.5V: R24.1, R?.1, R?.2
- new net +1.2V: R?.1
- new net +10V: U7.7 (V+)
- new net +12V: U?.7 (V+)
- new net -12V: U7.4 (V-), U?.4 (V-)
- new net ADC_IN_1: U?.6
- new net DAC_OUT_1: R21.2
Other:
- note added: "(-10V)-10V -> 0V-1V (Noninverting Amplifier with offset)"
- note added: "0V-1V -> (-10V)-10V (Difference Amplifier)"
- note added: "1.2V -> 0.5V"
- note added: ">1 Hz DC Block Filter"
- moved on the sheet: J10, J6

Commit message: improved pcb design
Parts:
- R15, R21, R23, R24, R25, R26: footprint (none) -> Resistor_SMD:R_0603_1608Metric
- R27, R28: renamed from R?; footprint (none) -> Resistor_SMD:R_0603_1608Metric
- gave numbers to parts that had none: 2
Other:
- note added: "NANOSURF = HIGH IMPEDANCE STM = LOW IMPEDANCE MAYBE ADD AN VOLTAGE FOLLOWER"
Changed lines of the file:
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@@
+		)
+	)
+	(text "NANOSURF = HIGH IMPEDANCE\nSTM = LOW IMPEDANCE\nMAYBE ADD AN VOLTAGE FOLLOWER\n"
+		(exclude_from_sim no)
+		(at 94.7077 82.8123 0)
+		(effects
+			(font
+				(size 1.27 1.27)
+			)
 		)
 	)
@@
 			)
 		)
-		(property "Footprint" ""
+		(property "Footprint" "Resistor_SMD:R_0603_1608Metric"
 			(at 164.338 74.93 90)
 			(effects
@@
 			)
 		)
-		(property "Footprint" ""
+		(property "Footprint" "Resistor_SMD:R_0603_1608Metric"
 			(at 158.75 66.802 90)
 			(effects
@@
 			)
 		)
-		(property "Footprint" ""
+		(property "Footprint" "Resistor_SMD:R_0603_1608Metric"
 			(at 255.27 74.168 90)
 			(effects
@@
 		(dnp no)
 		(fields_autoplaced yes)
-		(property "Reference" "R?"
+		(property "Reference" "R27"
 			(at 229.87 125.7299 0)
 			(effects
@@
 			)
 		)
-		(property "Footprint" ""
+		(property "Footprint" "Resistor_SMD:R_0603_1608Metric"
 			(at 225.552 127 90)
 			(effects
@@
 			(project ""
 				(path "/f8740766-88d0-4c4d-b661-742f36f22c7b/048a3674-481e-4b9e-b0e7-4786a4679f0c"
-					(reference "R?")
+					(reference "R27")
 					(unit 1)
 				)
@@
 		(dnp no)
 		(fields_autoplaced yes)
-		(property "Reference" "R?"
+		(property "Reference" "R28"
 			(at 237.49 74.9299 0)
 			(effects
@@
 			)
 		)
-		(property "Footprint" ""
+		(property "Footprint" "Resistor_SMD:R_0603_1608Metric"
 			(at 236.728 76.2 90)
 			(effects
@@
 			(project ""
 				(path "/f8740766-88d0-4c4d-b661-742f36f22c7b/048a3674-481e-4b9e-b0e7-4786a4679f0c"
-					(reference "R?")
+					(reference "R28")
 					(unit 1)
 				)
@@
 			)
 		)
-		(property "Footprint" ""
+		(property "Footprint" "Resistor_SMD:R_0603_1608Metric"
 			(at 226.568 67.31 90)
 			(effects
@@
 		(dnp no)
 		(fields_autoplaced yes)
-		(property "Reference" "U?"
+		(property "Reference" "U8"
 			(at 138.43 46.9198 0)
 			(effects
@@
 			(project ""
 				(path "/f8740766-88d0-4c4d-b661-742f36f22c7b/048a3674-481e-4b9e-b0e7-4786a4679f0c"
-					(reference "U?")
+					(reference "U8")
 					(unit 1)
 				)
@@
 			)
 		)
-		(property "Footprint" ""
+		(property "Footprint" "Resistor_SMD:R_0603_1608Metric"
 			(at 225.552 137.16 90)
 			(effects
@@
 		(dnp no)
 		(fields_autoplaced yes)
-		(property "Reference" "C?"
+		(property "Reference" "C33"
 			(at 58.42 60.9599 0)
 			(effects
@@
 			(project ""
 				(path "/f8740766-88d0-4c4d-b661-742f36f22c7b/048a3674-481e-4b9e-b0e7-4786a4679f0c"
-					(reference "C?")
+					(reference "C33")
 					(unit 1)
 				)
@@
 			)
 		)
-		(property "Footprint" ""
+		(property "Footprint" "Resistor_SMD:R_0603_1608Metric"
 			(at 220.98 59.182 90)
 			(effects
