File: hardware/synthesizer/microcontroller.kicad_sch (KiCad schematic)
At the start: 48 parts, among them U2 LAN8742A, U4 STM32H723VGT6, Y1 48MHz/8pF, Y3 32.768KHz/8pF

Commit message: further improvements
Parts:
- added SW2, SW3, SW?: RotaryEncoder, symbol Device:RotaryEncoder
- gave numbers to parts that had none: 4
Connections:
- net +3.3V: now also SW2.A, SW3.A, SW?.A
- net GND: now also SW2.B, SW3.B, SW?.B
Other:
- note added: "Rotary Encodrers"

Commit message: improved pcb design
Parts:
- D1, D2, D3: footprint (none) -> LED_SMD:LED_0201_0603Metric
- R1, R10, R11, R12, R16, R17, R18, R19, R2, R22, R7, R8, R9: footprint (none) -> Resistor_SMD:R_0603_1608Metric
- gave numbers to parts that had none: 1

Commit message: improved pcb design
Parts:
- C1, C18, C19, C2, C20, C25, C26, C27, C28, C29, C3, C32, C8: footprint (none) -> Capacitor_SMD:C_0603_1608Metric
- SW2, SW3, SW4: footprint (none) -> Rotary_Encoder:RotaryEncoder_Bourns_Horizontal_PEC09-2xxxF-Sxxxx

Commit message: add a lot of new stuff
Parts:
- removed SW2, SW3, SW4: RotaryEncoder, Rotary_Encoder:RotaryEncoder_Bourns_Horizontal_PEC09-2xxxF-Sxxxx, symbol Device:RotaryEncoder
- added J2: Conn_01x04_Socket, symbol Connector:Conn_01x04_Socket
Connections:
- net NSS: now reaches U4.28 (PA4)
- net NSS: now also J2.1 (Pin_1)
- net SCLK: now reaches U4.29 (PA5)
- net SCLK: now also J2.2 (Pin_2)
- net MISO: now reaches U4.30 (PA6)
- net MISO: now also J2.3 (Pin_3)
- net MOSI: now reaches U4.31 (PA7)
- net MOSI: now also J2.4 (Pin_4)
Other:
- note added: "SPI OUT"
- note removed: "Rotary Encodrers"
- moved on the sheet: C22, C30
