File: hardware/synthesizer/synthesizer.kicad_pcb (KiCad board)
At the start: 2 copper layers, 15 parts, among them J1 Conn_ARM_SWD_TagConnect_TC2030, J10 Output 2, J11 RJ45_Abracon_ARJP11A-MASA-B-A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, J6 Input 1, J7 Input 2, J9 Output 1, U1 MAX40200ANS, U2 LAN8742A, U3 AP2112K-1.2, U4 STM32H723VGT6, U5 AP2112K-3.3, U6 USBLC6-2P6, Y2 SG-210STF

Commit message: improved pcb design
Parts:
- added D1: Yellow, LED_SMD:LED_0201_0603Metric, F.Cu at (165.7, 93.0)
- added D2: Red, LED_SMD:LED_0201_0603Metric, F.Cu at (165.7, 94.8)
- added D3: Green, LED_SMD:LED_0201_0603Metric, F.Cu at (165.7, 96.5)
- added D6: Red, LED_SMD:LED_0201_0603Metric, F.Cu at (145.3, 95.7)
- added D8: Blue, LED_SMD:LED_0201_0603Metric, F.Cu at (145.3, 97.4)
- added D9: Orange, LED_SMD:LED_0201_0603Metric, F.Cu at (145.3, 99.2)
- added H1: MountingHole, MountingHole:MountingHole_2.2mm_M2_Pad, F.Cu at (218.9, 47.0)
- added H2: MountingHole, MountingHole:MountingHole_2.2mm_M2_Pad, F.Cu at (218.9, 115.0)
- added H3: MountingHole, MountingHole:MountingHole_2.2mm_M2_Pad, F.Cu at (85.0, 116.0)
- added H4: MountingHole, MountingHole:MountingHole_2.2mm_M2_Pad, F.Cu at (87.0, 50.0)
- added J8: USB_C_Receptacle_USB2.0_14P, Connector_USB:USB_C_Receptacle_HCTL_HC-TYPE-C-16P-01A, F.Cu at (99.7, 44.1)
- added R1: 1k, Resistor_SMD:R_0603_1608Metric, F.Cu at (163.2, 74.0)
- added R10: 10k, Resistor_SMD:R_0603_1608Metric, F.Cu at (167.2, 74.0)
- added R11: 10k, Resistor_SMD:R_0603_1608Metric, F.Cu at (167.2, 76.5)
- added R12: 5.6k, Resistor_SMD:R_0603_1608Metric, F.Cu at (167.2, 79.0)
- added R13: 1k, Resistor_SMD:R_0603_1608Metric, F.Cu at (141.8, 98.6)
- added R14: 1k, Resistor_SMD:R_0603_1608Metric, F.Cu at (141.8, 101.1)
- added R15: 200k, Resistor_SMD:R_0603_1608Metric, F.Cu at (141.8, 74.0)
- added R16: 100k, Resistor_SMD:R_0603_1608Metric, F.Cu at (167.2, 81.5)
- added R17: 1k, Resistor_SMD:R_0603_1608Metric, F.Cu at (167.2, 84.0)
- added R18: 10k, Resistor_SMD:R_0603_1608Metric, F.Cu at (171.2, 74.0)
- added R19: 49.9k, Resistor_SMD:R_0603_1608Metric, F.Cu at (171.2, 76.5)
- added R2: 1k, Resistor_SMD:R_0603_1608Metric, F.Cu at (163.2, 76.5)
- added R20: 470, Resistor_SMD:R_0603_1608Metric, F.Cu at (155.2, 102.3)
- added R21: 10k, Resistor_SMD:R_0603_1608Metric, F.Cu at (141.8, 76.5)
- added R22: 10k, Resistor_SMD:R_0603_1608Metric, F.Cu at (171.2, 79.0)
- added R23: 200k, Resistor_SMD:R_0603_1608Metric, F.Cu at (141.8, 79.0)
- added R24: 6.8k, Resistor_SMD:R_0603_1608Metric, F.Cu at (141.8, 81.5)
- added R25: 10k, Resistor_SMD:R_0603_1608Metric, F.Cu at (141.8, 84.0)
- added R26: 200k, Resistor_SMD:R_0603_1608Metric, F.Cu at (141.8, 86.5)
- added R27: 4.7k, Resistor_SMD:R_0603_1608Metric, F.Cu at (141.8, 89.0)
- added R28: 10k, Resistor_SMD:R_0603_1608Metric, F.Cu at (141.8, 91.5)
- added R3: 5.1k, Resistor_SMD:R_0603_1608Metric, F.Cu at (163.2, 98.7)
- added R4: 470, Resistor_SMD:R_0603_1608Metric, F.Cu at (155.2, 99.8)
- added R5: 5.1k, Resistor_SMD:R_0603_1608Metric, F.Cu at (163.2, 101.2)
- added R6: 1k, Resistor_SMD:R_0603_1608Metric, F.Cu at (141.8, 96.1)
- added R7: 49.9k, Resistor_SMD:R_0603_1608Metric, F.Cu at (163.2, 79.0)
- added R8: 49.9k, Resistor_SMD:R_0603_1608Metric, F.Cu at (163.2, 81.5)
- added R9: 49.9k, Resistor_SMD:R_0603_1608Metric, F.Cu at (163.2, 84.0)
- added U7: OPA196xDGK, Package_SO:VSSOP-8_3x3mm_P0.65mm, F.Cu at (147.5, 75.1)
- added U8: OPA196xDGK, Package_SO:VSSOP-8_3x3mm_P0.65mm, F.Cu at (147.5, 79.8)
- moved J6 83.3 mm to (201.0, 47.0)
- moved U2 72.2 mm to (210.3, 92.1), turned to 45 degrees
- moved J1 67.8 mm to (206.5, 80.0)
- moved D7 60.7 mm to (199.1, 104.0)
- moved U4 60.3 mm to (186.6, 92.4), turned to 45 degrees
- moved J7 54.7 mm to (183.0, 47.0)
- moved J10 48.4 mm to (142.1, 47.0)
- moved Y2 48.1 mm to (125.6, 104.5)
- moved F2 48.1 mm to (125.1, 94.2)
- moved U3 48.1 mm to (125.9, 83.7)
- moved U5 48.1 mm to (125.9, 88.3)
- moved U6 48.1 mm to (125.4, 98.9)
- moved J11 46.8 mm to (122.1, 60.0), turned to 180 degrees
- moved U1 43.4 mm to (135.8, 108.8)
- moved J9 36.2 mm to (160.0, 47.0)
Connections:
- J10 pad 1: unconnected-(J10-In-Pad1) -> /Coxial Connectors/OUT_2
- J6 pad 1: unconnected-(J6-In-Pad1) -> /Coxial Connectors/IN_1
- J7 pad 1: unconnected-(J7-In-Pad1) -> /Coxial Connectors/IN_2
- J9 pad 1: unconnected-(J9-In-Pad1) -> /Coxial Connectors/OUT_1
Other:
- board outline added: 151.1 x 81 mm

Commit message: improved pcb design
Parts:
- added C1: 100n/50V, Capacitor_SMD:C_0603_1608Metric, F.Cu at (203.7, 88.0)
- added C18: 100n/10V, Capacitor_SMD:C_0603_1608Metric, F.Cu at (203.7, 98.0)
- added C19: 100n/50V, Capacitor_SMD:C_0603_1608Metric, F.Cu at (207.7, 88.0)
- added C2: 100n/50V, Capacitor_SMD:C_0603_1608Metric, F.Cu at (203.7, 90.5)
- added C20: 100n/50V, Capacitor_SMD:C_0603_1608Metric, F.Cu at (207.7, 90.5)
- added C25: 100n/50V, Capacitor_SMD:C_0603_1608Metric, F.Cu at (207.7, 93.0)
- added C26: 100n/50V, Capacitor_SMD:C_0603_1608Metric, F.Cu at (207.7, 95.5)
- added C27: 100n/50V, Capacitor_SMD:C_0603_1608Metric, F.Cu at (207.7, 98.0)
- added C28: 10p/50V, Capacitor_SMD:C_0603_1608Metric, F.Cu at (211.7, 88.0)
- added C29: 10p/50V, Capacitor_SMD:C_0603_1608Metric, F.Cu at (211.7, 90.5)
- added C3: 100n/50V, Capacitor_SMD:C_0603_1608Metric, F.Cu at (203.7, 93.0)
- added C31: 100nF/10V, Capacitor_SMD:C_0603_1608Metric, F.Cu at (229.2, 74.0)
- added C32: 100n/50V, Capacitor_SMD:C_0603_1608Metric, F.Cu at (211.7, 93.0)
- added C8: 100n/50V, Capacitor_SMD:C_0603_1608Metric, F.Cu at (203.7, 95.5)
- added SW2: RotaryEncoder, Rotary_Encoder:RotaryEncoder_Bourns_Horizontal_PEC09-2xxxF-Sxxxx, F.Cu at (116.6, 114.5)
- added SW3: RotaryEncoder, Rotary_Encoder:RotaryEncoder_Bourns_Horizontal_PEC09-2xxxF-Sxxxx, F.Cu at (105.5, 114.5)
- added SW4: RotaryEncoder, Rotary_Encoder:RotaryEncoder_Bourns_Horizontal_PEC09-2xxxF-Sxxxx, F.Cu at (94.5, 114.5)
- added TP2: TestPoint, TestPoint:TestPoint_THTPad_1.0x1.0mm_Drill0.5mm, F.Cu at (228.7, 66.2)
- added TP3: TestPoint, TestPoint:TestPoint_THTPad_1.0x1.0mm_Drill0.5mm, F.Cu at (228.7, 69.2)
- moved U2 86.2 mm to (128.3, 65.5)
- moved J10 74.3 mm to (174.0, 114.0), turned to 180 degrees
- moved J1 71.9 mm to (137.5, 59.5)
- moved J9 67.1 mm to (156.0, 114.0), turned to 180 degrees
- moved U1 55.9 mm to (91.2, 75.2)
- moved R3 35.2 mm to (135.0, 77.5)
- moved R5 35.2 mm to (135.0, 80.0)
- moved R11 34.0 mm to (135.8, 89.5)
- moved R17 34.0 mm to (135.8, 97.0)
- moved R2 34.0 mm to (131.8, 89.5)
- moved R9 34.0 mm to (131.8, 97.0)
- moved R1 34.0 mm to (131.8, 87.0)
- moved R10 34.0 mm to (135.8, 87.0)
- moved R12 34.0 mm to (135.8, 92.0)
- moved R16 34.0 mm to (135.8, 94.5)
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Other:
- board size 151.1 x 81 mm -> 117.2 x 81 mm

Commit message: add a lot of new stuff
Parts:
- moved C31 59.9 mm to (169.5, 69.8)
- moved TP2 59.9 mm to (169.0, 62.0)
- moved TP3 59.9 mm to (169.0, 65.0)
- moved C18 29.9 mm to (179.8, 80.0)
- moved C2 29.9 mm to (179.8, 72.5)
- moved C29 29.9 mm to (187.8, 72.5)
- moved C1 29.9 mm to (179.8, 70.0)
- moved C28 29.9 mm to (187.8, 70.0)
- moved C3 29.9 mm to (179.8, 75.0)
- moved C32 29.9 mm to (187.8, 75.0)
- moved C8 29.9 mm to (179.8, 77.5)
- moved C20 29.9 mm to (183.8, 72.5)
- moved C27 29.9 mm to (183.8, 80.0)
- moved C19 29.9 mm to (183.8, 70.0)
- moved C25 29.9 mm to (183.8, 75.0)
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Changed lines of the file:
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@@
 			(psa4output no)
 			(plot_black_and_white yes)
-			(plotinvisibletext no)
 			(sketchpadsonfab no)
 			(plotpadnumbers no)
@@
 	(footprint "Resistor_SMD:R_0603_1608Metric"
 		(layer "F.Cu")
-		(at 113.4025 72.715)
+		(at 118.29 82.74)
 		(descr "Resistor SMD 0603 (1608 Metric), square (rectangular) end terminal, IPC_7351 nominal, (Body size source: IPC-SM-782 page 72, https://www.pcb-3d.com/wordpress/wp-content/uploads/ipc-sm-782a_amendment_1_and_2.pdf), generated with kicad-footprint-generator")
 		(tags "resistor")
@@
 	(footprint "Capacitor_SMD:C_0603_1608Metric"
 		(layer "F.Cu")
-		(at 203.655 98.04)
+		(at 179.765 80.02)
 		(descr "Capacitor SMD 0603 (1608 Metric), square (rectangular) end terminal, IPC_7351 nominal, (Body size source: IPC-SM-782 page 76, https://www.pcb-3d.com/wordpress/wp-content/uploads/ipc-sm-782a_amendment_1_and_2.pdf), generated with kicad-footprint-generator")
 		(tags "capacitor")
@@
 	(footprint "Package_SO:VSSOP-8_3x3mm_P0.65mm"
 		(layer "F.Cu")
-		(at 119.1125 71.325)
+		(at 124 81.35)
 		(descr "VSSOP, 8 Pin (https://www.jedec.org/standards-documents/docs/mo-187-f), generated with kicad-footprint-generator ipc_gullwing_generator.py")
 		(tags "VSSOP SO JEDEC-MO-187-AA TI-DGK0008A")
@@
 	(footprint "Capacitor_SMD:C_0603_1608Metric"
 		(layer "F.Cu")
-		(at 207.665 93.02)
+		(at 183.775 75)
 		(descr "Capacitor SMD 0603 (1608 Metric), square (rectangular) end terminal, IPC_7351 nominal, (Body size source: IPC-SM-782 page 76, https://www.pcb-3d.com/wordpress/wp-content/uploads/ipc-sm-782a_amendment_1_and_2.pdf), generated with kicad-footprint-generator")
 		(tags "capacitor")
@@
 	(footprint "Capacitor_SMD:C_0603_1608Metric"
 		(layer "F.Cu")
-		(at 207.665 88)
+		(at 183.775 69.98)
 		(descr "Capacitor SMD 0603 (1608 Metric), square (rectangular) end terminal, IPC_7351 nominal, (Body size source: IPC-SM-782 page 76, https://www.pcb-3d.com/wordpress/wp-content/uploads/ipc-sm-782a_amendment_1_and_2.pdf), generated with kicad-footprint-generator")
 		(tags "capacitor")
@@
 	(footprint "TestPoint:TestPoint_THTPad_1.0x1.0mm_Drill0.5mm"
 		(layer "F.Cu")
-		(at 228.745 66.17)
+		(at 169 61.95)
 		(descr "THT rectangular pad as test Point, square 1.0mm side length, hole diameter 0.5mm")
 		(tags "test point THT pad rectangle square")
@@
 	(footprint "Capacitor_SMD:C_0603_1608Metric"
 		(layer "F.Cu")
-		(at 211.675 88)
+		(at 187.785 69.98)
 		(descr "Capacitor SMD 0603 (1608 Metric), square (rectangular) end terminal, IPC_7351 nominal, (Body size source: IPC-SM-782 page 76, https://www.pcb-3d.com/wordpress/wp-content/uploads/ipc-sm-782a_amendment_1_and_2.pdf), generated with kicad-footprint-generator")
 		(tags "capacitor")
@@
 	(footprint "Capacitor_SMD:C_0603_1608Metric"
 		(layer "F.Cu")
-		(at 203.655 90.51)
+		(at 179.765 72.49)
 		(descr "Capacitor SMD 0603 (1608 Metric), square (rectangular) end terminal, IPC_7351 nominal, (Body size source: IPC-SM-782 page 76, https://www.pcb-3d.com/wordpress/wp-content/uploads/ipc-sm-782a_amendment_1_and_2.pdf), generated with kicad-footprint-generator")
 		(tags "capacitor")
@@
 		(tags "SMD SMT crystal oscillator")
 		(property "Reference" "Y2"
-			(at -20.65 -25.85 0)
+			(at -8.85 -1.65 0)
 			(layer "F.SilkS")
 			(effects
@@
 		)
 		(fp_text user "${REFERENCE}"
-			(at -20.65 -23.65 0)
+			(at -8.85 0.55 0)
 			(layer "F.Fab")
 			(effects
@@
 	(footprint "Capacitor_SMD:C_0603_1608Metric"
 		(layer "F.Cu")
-		(at 229.225 74)
+		(at 169.48 69.78)
 		(descr "Capacitor SMD 0603 (1608 Metric), square (rectangular) end terminal, IPC_7351 nominal, (Body size source: IPC-SM-782 page 76, https://www.pcb-3d.com/wordpress/wp-content/uploads/ipc-sm-782a_amendment_1_and_2.pdf), generated with kicad-footprint-generator")
 		(tags "capacitor")
@@
 	(footprint "Resistor_SMD:R_0603_1608Metric"
 		(layer "F.Cu")
-		(at 113.4025 70.205)
+		(at 118.29 80.23)
 		(descr "Resistor SMD 0603 (1608 Metric), square (rectangular) end terminal, IPC_7351 nominal, (Body size source: IPC-SM-782 page 72, https://www.pcb-3d.com/wordpress/wp-content/uploads/ipc-sm-782a_amendment_1_and_2.pdf), generated with kicad-footprint-generator")
 		(tags "resistor")
@@
 	(footprint "Capacitor_SMD:C_0603_1608Metric"
 		(layer "F.Cu")
-		(at 203.655 95.53)
+		(at 179.765 77.51)
 		(descr "Capacitor SMD 0603 (1608 Metric), square (rectangular) end terminal, IPC_7351 nominal, (Body size source: IPC-SM-782 page 76, https://www.pcb-3d.com/wordpress/wp-content/uploads/ipc-sm-782a_amendment_1_and_2.pdf), generated with kicad-footprint-generator")
 		(tags "capacitor")
@@
 	(footprint "Resistor_SMD:R_0603_1608Metric"
 		(layer "F.Cu")
-		(at 113.4025 75.225)
+		(at 118.29 85.25)
 		(descr "Resistor SMD 0603 (1608 Metric), square (rectangular) end terminal, IPC_7351 nominal, (Body size source: IPC-SM-782 page 72, https://www.pcb-3d.com/wordpress/wp-content/uploads/ipc-sm-782a_amendment_1_and_2.pdf), generated with kicad-footprint-generator")
 		(tags "resistor")
@@
 	(footprint "Capacitor_SMD:C_0603_1608Metric"
 		(layer "F.Cu")
-		(at 203.655 88)
+		(at 179.765 69.98)
 		(descr "Capacitor SMD 0603 (1608 Metric), square (rectangular) end terminal, IPC_7351 nominal, (Body size source: IPC-SM-782 page 76, https://www.pcb-3d.com/wordpress/wp-content/uploads/ipc-sm-782a_amendment_1_and_2.pdf), generated with kicad-footprint-generator")
 		(tags "capacitor")
@@
 	(footprint "Package_DFN_QFN:VQFN-24-1EP_4x4mm_P0.5mm_EP2.5x2.5mm_ThermalVias"
 		(layer "F.Cu")
-		(at 128.253903 65.513864 45)
+		(at 116.292893 69.292893 45)
 		(descr "VQFN, 24 Pin (https://ww1.microchip.com/downloads/aemDocuments/documents/product-documents/package-drawings/24L-VQFN%E2%80%934x4x0.9mm-MJ-C04-00143b.pdf), generated with kicad-footprint-generator ipc_noLead_generator.py")
 		(tags "VQFN NoLead")
@@
 	(footprint "Capacitor_SMD:C_0603_1608Metric"
 		(layer "F.Cu")
-		(at 211.675 90.51)
+		(at 187.785 72.49)
 		(descr "Capacitor SMD 0603 (1608 Metric), square (rectangular) end terminal, IPC_7351 nominal, (Body size source: IPC-SM-782 page 76, https://www.pcb-3d.com/wordpress/wp-content/uploads/ipc-sm-782a_amendment_1_and_2.pdf), generated with kicad-footprint-generator")
 		(tags "capacitor")
@@
 	(footprint "Capacitor_SMD:C_0603_1608Metric"
 		(layer "F.Cu")
-		(at 207.665 95.53)
+		(at 183.775 77.51)
 		(descr "Capacitor SMD 0603 (1608 Metric), square (rectangular) end terminal, IPC_7351 nominal, (Body size source: IPC-SM-782 page 76, https://www.pcb-3d.com/wordpress/wp-content/uploads/ipc-sm-782a_amendment_1_and_2.pdf), generated with kicad-footprint-generator")
 		(tags "capacitor")
@@
 	(footprint "Resistor_SMD:R_0603_1608Metric"
 		(layer "F.Cu")
-		(at 113.4025 77.735)
+		(at 118.29 87.76)
 		(descr "Resistor SMD 0603 (1608 Metric), square (rectangular) end terminal, IPC_7351 nominal, (Body size source: IPC-SM-782 page 72, https://www.pcb-3d.com/wordpress/wp-content/uploads/ipc-sm-782a_amendment_1_and_2.pdf), generated with kicad-footprint-generator")
 		(tags "resistor")
@@
 	(footprint "TestPoint:TestPoint_THTPad_1.0x1.0mm_Drill0.5mm"
 		(layer "F.Cu")
-		(at 228.745 69.22)
+		(at 169 65)
 		(descr "THT rectangular pad as test Point, square 1.0mm side length, hole diameter 0.5mm")
 		(tags "test point THT pad rectangle square")
@@
 	(footprint "Capacitor_SMD:C_0603_1608Metric"
 		(layer "F.Cu")
-		(at 207.665 98.04)
+		(at 183.775 80.02)
 		(descr "Capacitor SMD 0603 (1608 Metric), square (rectangular) end terminal, IPC_7351 nominal, (Body size source: IPC-SM-782 page 76, https://www.pcb-3d.com/wordpress/wp-content/uploads/ipc-sm-782a_amendment_1_and_2.pdf), generated with kicad-footprint-generator")
 		(tags "capacitor")
@@
 	(footprint "Package_SO:VSSOP-8_3x3mm_P0.65mm"
 		(layer "F.Cu")
-		(at 119.1125 75.975)
+		(at 124 86)
 		(descr "VSSOP, 8 Pin (https://www.jedec.org/standards-documents/docs/mo-187-f), generated with kicad-footprint-generator ipc_gullwing_generator.py")
 		(tags "VSSOP SO JEDEC-MO-187-AA TI-DGK0008A")
@@
 	(footprint "Capacitor_SMD:C_0603_1608Metric"
 		(layer "F.Cu")
-		(at 211.675 93.02)
+		(at 187.785 75)
 		(descr "Capacitor SMD 0603 (1608 Metric), square (rectangular) end terminal, IPC_7351 nominal, (Body size source: IPC-SM-782 page 76, https://www.pcb-3d.com/wordpress/wp-content/uploads/ipc-sm-782a_amendment_1_and_2.pdf), generated with kicad-footprint-generator")
 		(tags "capacitor")
@@
 	(footprint "Capacitor_SMD:C_0603_1608Metric"
 		(layer "F.Cu")
-		(at 203.655 93.02)
+		(at 179.765 75)
 		(descr "Capacitor SMD 0603 (1608 Metric), square (rectangular) end terminal, IPC_7351 nominal, (Body size source: IPC-SM-782 page 76, https://www.pcb-3d.com/wordpress/wp-content/uploads/ipc-sm-782a_amendment_1_and_2.pdf), generated with kicad-footprint-generator")
 		(tags "capacitor")
@@
 	(footprint "Capacitor_SMD:C_0603_1608Metric"
 		(layer "F.Cu")
-		(at 207.665 90.51)
+		(at 183.775 72.49)
 		(descr "Capacitor SMD 0603 (1608 Metric), square (rectangular) end terminal, IPC_7351 nominal, (Body size source: IPC-SM-782 page 76, https://www.pcb-3d.com/wordpress/wp-content/uploads/ipc-sm-782a_amendment_1_and_2.pdf), generated with kicad-footprint-generator")
 		(tags "capacitor")
